File: fpaa_esp32_badge/leds.kicad_sch (KiCad schematic)
At the start: 37 parts, among them J12 Conn_01x02, J13 Conn_01x02, J14 Conn_01x02

Commit message: added pdf and corrected some part values
Parts:
- R20, R21: value R -> 82
- R5: value R -> 180
Changed lines of the file:
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@@
       (effects (font (size 1.27 1.27)) (justify left))
     )
-    (property "Value" "R" (at 66.04 114.3 0)
+    (property "Value" "82" (at 66.04 114.3 0)
       (effects (font (size 1.27 1.27)) (justify left))
     )
@@
       (effects (font (size 1.27 1.27)) (justify left))
     )
-    (property "Value" "R" (at 88.9 114.3 0)
+    (property "Value" "82" (at 88.9 114.3 0)
       (effects (font (size 1.27 1.27)) (justify left))
     )
@@
       (effects (font (size 1.27 1.27)) (justify left))
     )
-    (property "Value" "R" (at 41.91 114.3 0)
-      (effects (font (size 1.27 1.27)) (justify left))
-    )
+    (property "Value" "180" (at 41.91 114.3 0)
+      (effects (font (size 1.27 1.27)) (justify left))
+    )
