File: fpaa_esp32_badge/fpaa_esp32_badge.kicad_pcb (KiCad board)
At the start: 4 copper layers, 99.1 x 99.1 mm, 233 parts, among them J1 Conn_01x04, J10 AudioPlug3, J11 Conn_01x05, J12 Conn_01x02, J13 Conn_01x02, J14 Conn_01x02, J16 Conn_01x12, J17 Conn_01x01, J18 Conn_01x01, J19 Conn_01x01, J2 Conn_01x04, J20 AudioPlug3, J21 Conn_01x02, J22 Conn_01x03, J23 Conn_01x02, J3 Conn_01x04, J4 Conn_01x04, J5 USB_C_Receptacle_USB2.0, J6 Micro_SD_Card_Det1, J7 Conn_Coaxial, J8 Conn_Coaxial, J9 Conn_Coaxial, SW1 SW_Push, SW2 SW_Push, SW3 SW_Push, T10 Transformer_1P_1S, T11 Transformer_1P_1S, T9 Transformer_1P_1S, U10 LT6350IMS8_PBF, U11 PCM5102, U2 ESP32-S3-WROOM-1, U3 AMS1117-3.3, U4 AZ1117-3.3, U5 LM324, U6 LM324, U7 LT6350IMS8_PBF, U8 LT6350IMS8_PBF, U9 LT6350IMS8_PBF, X1 SG-5032CAN

Commit message: Updated html bom with all values
Parts:
- C43, C44, C45, C46: value C -> 2.2uF
- R20, R21: value R -> 82
- R5: value R -> 180
- R85: value R -> 1K
Changed lines of the file:
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@@
         (effects (font (size 1 1) (thickness 0.15)))
     )
-    (fp_text value "C" (at 0 1.43 90) (layer "F.Fab")
+    (fp_text value "2.2uF" (at 0 1.43 90) (layer "F.Fab")
         (effects (font (size 1 1) (thickness 0.15)))
     )
@@
         (effects (font (size 1 1) (thickness 0.15)))
     )
-    (fp_text value "C" (at 0 1.43) (layer "F.Fab")
+    (fp_text value "2.2uF" (at 0 1.43) (layer "F.Fab")
         (effects (font (size 1 1) (thickness 0.15)))
     )
@@
         (effects (font (size 1 1) (thickness 0.15)))
     )
-    (fp_text value "C" (at 0 1.43 90) (layer "F.Fab")
+    (fp_text value "2.2uF" (at 0 1.43 90) (layer "F.Fab")
         (effects (font (size 1 1) (thickness 0.15)))
     )
@@
         (effects (font (size 1 1) (thickness 0.15)))
     )
-    (fp_text value "C" (at 0 1.43 90) (layer "F.Fab")
+    (fp_text value "2.2uF" (at 0 1.43 90) (layer "F.Fab")
         (effects (font (size 1 1) (thickness 0.15)))
     )
@@
         (effects (font (size 1 1) (thickness 0.15)))
     )
-    (fp_text value "R" (at 0.051701 1.464001 90) (layer "F.Fab")
+    (fp_text value "1K" (at 0.051701 1.464001 90) (layer "F.Fab")
         (effects (font (size 1 1) (thickness 0.15)))
     )
@@
         (effects (font (size 1 1) (thickness 0.15)) (justify mirror))
     )
-    (fp_text value "R" (at 0 -1.43 90) (layer "B.Fab")
+    (fp_text value "82" (at 0 -1.43 90) (layer "B.Fab")
         (effects (font (size 1 1) (thickness 0.15)) (justify mirror))
     )
@@
         (effects (font (size 1 1) (thickness 0.15)) (justify mirror))
     )
-    (fp_text value "R" (at 0 -1.43 90) (layer "B.Fab")
+    (fp_text value "82" (at 0 -1.43 90) (layer "B.Fab")
         (effects (font (size 1 1) (thickness 0.15)) (justify mirror))
     )
@@
         (effects (font (size 1 1) (thickness 0.15)) (justify mirror))
     )
-    (fp_text value "R" (at 0 -1.43 90) (layer "B.Fab")
+    (fp_text value "180" (at 0 -1.43 90) (layer "B.Fab")
         (effects (font (size 1 1) (thickness 0.15)) (justify mirror))
     )
